File: KVM_Switch.kicad_sch (KiCad schematic)
At the start: 0 parts

Commit message: Publish A2 hardware, firmware, and verification package
Other:
- note added: "12V DC input 5V buck supply for four USB ports 3.3V logic supply Reverse-polarity protection"
- note added: "Four USB 2.0 peripheral ports Self-powered hub Individual current-limited port switches USB ESD protection"
- note added: "Push button selects computer 1 or 2 Video and USB disconnect before selection changes Host USB VBUS sensing SWD programming header"
- note added: "Two HDMI inputs per computer Two independently extended HDMI monitors Two USB-C data-only upstream ports External USB-C to HDMI adapter per laptop No charging or EDID emulation"
- title: KVM Switch — Top Level -> Two-computer HDMI and USB switch
Changed lines of the file:
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@@
 	(paper "A4")
 	(title_block
-		(title "KVM Switch — Top Level")
-		(rev "1.0")
+		(title "Two-computer HDMI and USB switch")
+		(date "2026-09-06")
+		(rev "A2")
+		(comment 1 "Routed prototype - hardware validation required")
+	)
+	(text "Four USB 2.0 peripheral ports\nSelf-powered hub\nIndividual current-limited port switches\nUSB ESD protection"
+		(exclude_from_sim no)
+		(at 205 135 0)
+		(effects
+			(font
+				(size 1.27 1.27)
+			)
+		)
+	)
+	(text "Two HDMI inputs per computer\nTwo independently extended HDMI monitors\nTwo USB-C data-only upstream ports\nExternal USB-C to HDMI adapter per laptop\nNo charging or EDID emulation"
+		(exclude_from_sim no)
+		(at 72 135 0)
+		(effects
+			(font
+				(size 1.27 1.27)
+			)
+		)
+	)
+	(text "Push button selects computer 1 or 2\nVideo and USB disconnect before selection changes\nHost USB VBUS sensing\nSWD programming header"
+		(exclude_from_sim no)
+		(at 205 50 0)
+		(effects
+			(font
+				(size 1.27 1.27)
+			)
+		)
+	)
+	(text "12V DC input\n5V buck supply for four USB ports\n3.3V logic supply\nReverse-polarity protection"
+		(exclude_from_sim no)
+		(at 72 50 0)
+		(effects
+			(font
+				(size 1.27 1.27)
+			)
+		)
 	)
 	(sheet
