File: sheet_hub.kicad_sch  .kicad_sch (KiCad schematic)
At the start: 26 parts, among them U10 USB2514B_M2, U9 TS3USB221RSERG4, Y1 Crystal

Commit message: Publish A2 hardware, firmware, and verification package
Parts:
- removed F1, F2, F3, F4: BSMD1206-050-6V, polyfuse:F1206, symbol polyfuse:BSMD1206-050-6V
- removed J_USB1, J_USB2, J_USB3, J_USB4: KH-3.0USB-AM-9P, usb_a_connector:USB-3.0-SMD_KH-3.0USB-AM-9P, symbol usb_a_connector:KH-3.0USB-AM-9P
- removed R5: 1M, Resistor_SMD:R_0402_1005Metric, symbol Device:R
- removed Y1: Crystal, Crystal:Crystal_SMD_3225-4Pin_3.2x2.5mm, symbol Device:Crystal
- added C26: 1uF, Capacitor_SMD:C_0603_1608Metric, symbol Device:C
- added C34, C35, C36, C37, C38, C39, C40, C41, C42: 100nF, Capacitor_SMD:C_0402_1005Metric, symbol Device:C
- added C43, C44, C45, C46: 220uF, Capacitor_SMD:CP_Elec_6.3x7.7, symbol Device:C_Polarized
- added J_USB1: USB1046-GF-0190-L-B-A, KVM_Custom_Footprints:Assembly_J_USB1, symbol KVM_Custom:USB1046_USB2
- added J_USB2: USB1046-GF-0190-L-B-A, KVM_Custom_Footprints:Assembly_J_USB2, symbol KVM_Custom:USB1046_USB2
- added J_USB3: USB1046-GF-0190-L-B-A, KVM_Custom_Footprints:Assembly_J_USB3, symbol KVM_Custom:USB1046_USB2
- added J_USB4: USB1046-GF-0190-L-B-A, KVM_Custom_Footprints:Assembly_J_USB4, symbol KVM_Custom:USB1046_USB2
- added R25, R26, R27, R28, R29, R30, R31, R32, R33: 100k, Resistor_SMD:R_0402_1005Metric, symbol Device:R
- added R39, R40, R41, R42: 10k, Resistor_SMD:R_0402_1005Metric, symbol Device:R
- added U20, U21, U22, U23: TPS2051CDBVR, Package_TO_SOT_SMD:SOT-23-5, symbol Power_Management:TPS2051CDBV
- added Y1: 24MHz 12pF, KVM_Custom_Footprints:Assembly_Y1, symbol Device:Crystal_GND24
- C18: value 1uF -> 100nF; footprint Capacitor_SMD:C_0402_1005Metric -> Capacitor_SMD:C_0603_1608Metric; Dielectric (none) -> X7R; LCSC Part (none) -> C14663; MPN (none) -> CC0603KRX7R9BB104; Manufacturer (none) -> YAGEO; Voltage (none) -> 50V
- C19, C20: value 22pF -> 18pF; Dielectric (none) -> C0G; LCSC Part (none) -> C76701; MPN (none) -> CGA2B2C0G1H180JT0Y0F; Manufacturer (none) -> TDK; Voltage (none) -> 50V
- C21: value 1uF -> 100nF; Dielectric (none) -> X7R; LCSC Part (none) -> C131394; MPN (none) -> CC0402KRX7R9BB104; Manufacturer (none) -> YAGEO; Voltage (none) -> 50V
- C22, C25: value 0.1uF -> 100nF; Dielectric (none) -> X7R; LCSC Part (none) -> C131394; MPN (none) -> CC0402KRX7R9BB104; Manufacturer (none) -> YAGEO; Voltage (none) -> 50V
- C23: footprint Capacitor_SMD:C_0603_1608Metric -> Capacitor_SMD:C_0805_2012Metric; Dielectric (none) -> X7R; LCSC Part (none) -> C95841; MPN (none) -> CL21B106KOQNNNE; Manufacturer (none) -> Samsung Electro-Mechanics; Voltage (none) -> 16V
- C24: footprint Capacitor_SMD:C_0402_1005Metric -> Capacitor_SMD:C_0603_1608Metric; Dielectric (none) -> X7R; LCSC Part (none) -> C59782; MPN (none) -> CL10B105KO8NNNC; Manufacturer (none) -> Samsung Electro-Mechanics; Voltage (none) -> 16V
- D1, D2, D3, D4: Manufacturer ST(意法半导体) -> (none)
- R12: LCSC Part (none) -> C11692; MPN (none) -> 0402WGF1242TCE; Manufacturer (none) -> UNI-ROYAL; Power (none) -> 62.5mW; Tolerance (none) -> 1%
- R13: LCSC Part (none) -> C25744; MPN (none) -> 0402WGF1002TCE; Manufacturer (none) -> UNI-ROYAL; Power (none) -> 62.5mW; Tolerance (none) -> 1%
- U10: value USB2514B_M2 -> USB2514B-AEZC-TR; footprint Package_DFN_QFN:Texas_RHH0036C_VQFN-36-1EP_6x6mm_P0.5mm_EP4.4x4.4mm_ThermalVias -> Package_DFN_QFN:QFN-36-1EP_6x6mm_P0.5mm_EP3.7x3.7mm_ThermalVias; Availability Not in stock -> (none); Check_prices https://www.snapeda.com/parts/USB2514B/M2/Microchip+Technol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 -> (none); LCSC Part (none) -> C16251; MF Microchip -> (none); MP USB2514B/M2 -> (none); MPN (none) -> USB2514B-AEZC-TR; Package VFQFN-36 Microchip -> (none); Price None -> (none); SnapEDA_Link https://www.snapeda.com/parts/USB2514B/M2/Microchip+Technol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 -> (none)
- U9: value TS3USB221RSERG4 -> TS3USB221RSER; footprint Package_TO_SOT_SMD:SOT-23-8 -> Package_DFN_QFN:Texas_UQFN-10_1.5x2mm_P0.5mm; Availability In Stock -> (none); Check_prices https://www.snapeda.com/parts/TS3USB221RSERG4/Texas+Instrum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 -> (none); LCSC Part (none) -> C130085; MF Texas Instruments -> (none); MP TS3USB221RSERG4 -> (none); MPN (none) -> TS3USB221RSER; Manufacturer (none) -> Texas Instruments; Package UQFN-10 Texas Instruments -> (none); Price None -> (none); SnapEDA_Link https://www.snapeda.com/parts/TS3USB221RSERG4/Texas+Instrum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 -> (none)
Connections:
- net USB1_DM is gone; now on net USB_D1_N: D1.6
- net USB1_DP is gone; now on net USB_D1_P: D1.4
- net USB2_DM is gone; now on net USB_D2_N: D2.6
- net USB2_DP is gone; now on net USB_D2_P: D2.4
- net USB3_DM is gone; now on net USB_D3_N: D3.6
- net USB3_DP is gone; now on net USB_D3_P: D3.4
- net USB4_DM is gone; now on net USB_D4_N: D4.6
- net USB4_DP is gone; now on net USB_D4_P: D4.4
- net +3.3V: now also C22.1, C23.1, C24.1, C25.1, U9.10 (VCC), C26.1, C34.1, C35.1, C36.1, C37.1, C38.1, R25.1, R39.1, R40.1, R41.1, R42.1; no longer C22.2, C23.2, C24.2, C25.2, U10.27 (VBUS_DET)
- net +5V: now also C39.1, C40.1, C41.1, C42.1, U20.5 (IN), U21.5 (IN), U22.5 (IN), U23.5 (IN); no longer D1.5, D2.5, D3.5, D4.5
- net GND: now also C18.2, C19.2, C21.2, C22.2, C23.2, C24.2, C25.2, R12.2, C26.2, C34.2, C35.2, C36.2, C37.2, C38.2, C39.2, C40.2, C41.2, C42.2, C43.2, C44.2, C45.2, C46.2, J_USB1.4 (GND), J_USB1.SH (Shield), J_USB2.4 (GND), J_USB2.SH (Shield), J_USB3.4 (GND), J_USB3.SH (Shield), J_USB4.4 (GND), J_USB4.SH (Shield), R26.2, R27.2, R28.2, R29.2, R30.2, R31.2, R32.2, R33.2, U20.2 (GND), U21.2 (GND), U22.2 (GND), U23.2 (GND), Y1.2 (G), Y1.4 (G); no longer C18.1, C19.1, C21.1, C22.1, C23.1, C24.1, R12.1, U10.25 (CFG_SEL1), U9.6 (OE)
- net USB_D1_N: now also J_USB1.2 (D-)
- net USB_D1_P: now also J_USB1.3 (D+)
- net USB_D2_N: now also J_USB2.2 (D-)
- net USB_D2_P: now also J_USB2.3 (D+)
- net USB_D3_N: now also J_USB3.2 (D-)
- net USB_D3_P: now also J_USB3.3 (D+)
- net USB_D4_N: now also J_USB4.2 (D-)
- net USB_D4_P: now also J_USB4.3 (D+)
- net HUB_XTAL1: now reaches U10.32 (XTAL1)
- net HUB_XTAL1: now also C19.1, Y1.1; no longer C19.2
- net HUB_XTAL2: now reaches C20.1, U10.33 (XTAL2)
- net HUB_XTAL2: now also Y1.3
- net USB_PWR1: now reaches U10.12 (PRTPWR1)
- net USB_PWR1: now also R30.1, U20.4 (EN)
- net USB_OC1_N: now reaches U10.13 (OCS1)
- net USB_OC1_N: now also R39.2, U20.3 (~{FLT})
- net HUB_CRFILT: now reaches U10.14 (CRFILT)
- net HUB_CRFILT: now also C21.1; no longer C21.2
- net USB_PWR2: now reaches U10.16 (PRTPWR2)
- net USB_PWR2: now also R31.1, U21.4 (EN)
- net USB_OC2_N: now reaches U10.17 (OCS2)
- net USB_OC2_N: now also R40.2, U21.3 (~{FLT})
- net USB_PWR3: now reaches U10.18 (PRTPWR3)
- net USB_PWR3: now also R32.1, U22.4 (EN)
- net USB_OC3_N: now reaches U10.19 (OCS3)
- net USB_OC3_N: now also R41.2, U22.3 (~{FLT})
- net USB_PWR4: now reaches U10.20 (PRTPWR4)
- net USB_PWR4: now also R33.1, U23.4 (EN)
- net USB_OC4_N: now reaches U10.21 (OCS4)
- net USB_OC4_N: now also R42.2, U23.3 (~{FLT})
- net HUB_NONREM1: now reaches U10.22 (SMBDATA)
- net HUB_NONREM1: now also R29.1
- net HUB_CFG0: now reaches U10.24 (SMBCLK)
- net HUB_CFG0: now also R26.1
- net HUB_RESET_N: now reaches R13.2, U10.26 (~{RESET})
- net HUB_NONREM0: now reaches U10.28 (SUSP_IND)
- net HUB_NONREM0: now also R28.1
- net USB_UP_N: now reaches U10.30 (DM-UP), U9.7 (D_)
- net USB_UP_P: now reaches U10.31 (DP-UP), U9.8 (D+)
- net HUB_PLLFILT: now reaches U10.34 (PLLFILT)
- net HUB_PLLFILT: now also C18.1; no longer C18.2
- net HUB_RBIAS: now reaches U10.35 (RBIAS)
- net HUB_RBIAS: now also R12.1; no longer R12.2
- net USB2_DN_A renamed USB_HOST1_N
- net USB2_DN_B renamed USB_HOST2_N
- net USB2_DP_A renamed USB_HOST1_P
- net USB2_DP_B renamed USB_HOST2_P
- new net HUB_CFG1: R27.1, U10.25 (CFG_SEL1)
- new net HUB_VBUS_DET: U10.27 (VBUS_DET)
- new net USB_OE_N: R25.2, U9.6 (OE)
- new net USB_VBUS1: C43.1, D1.5, J_USB1.1 (VBUS), U20.1 (OUT)
- new net USB_VBUS2: C44.1, D2.5, J_USB2.1 (VBUS), U21.1 (OUT)
- new net USB_VBUS3: C45.1, D3.5, J_USB3.1 (VBUS), U22.1 (OUT)
- new net USB_VBUS4: C46.1, D4.5, J_USB4.1 (VBUS), U23.1 (OUT)
- no-connect marks 27 -> 0
Other:
- note added: "USB 2.0 self-powered hub: individual 500mA port switches and fault feedback. CFG[1:0]=00, all ports removable. No EEPROM required. VBUS_DET and upstream OE follow the selected host via MCU firmware. One 100nF at each hub supply pin; 18pF crystal loads require prototype verification."
- title: (none) -> Two-computer HDMI and USB switch
