File: sheet_pdn.kicad_sch (KiCad schematic)
At the start: 14 parts, among them J3 Conn_01x02, U1 TLV62569DBV, U2 AP2112K-3.3

Commit message: Publish A2 hardware, firmware, and verification package
Parts:
- removed J3: Conn_01x02, Connector_BarrelJack:BarrelJack_Horizontal, symbol Connector_Generic:Conn_01x02
- removed L2: 600R@100MHz, Inductor_SMD:L_0805_2012Metric, symbol Device:L
- removed U1: TLV62569DBV, Package_TO_SOT_SMD:SOT-23-5, symbol Regulator_Switching:TLV62569DBV
- added C16, C30: 10uF, Capacitor_SMD:C_1206_3216Metric, symbol Device:C
- added C31: 100nF, Capacitor_SMD:C_0402_1005Metric, symbol Device:C
- added C32: 1uF, Capacitor_SMD:C_0603_1608Metric, symbol Device:C
- added C33: 150pF, Capacitor_SMD:C_0402_1005Metric, symbol Device:C
- added C51, C52: 22uF, Capacitor_SMD:C_1206_3216Metric, symbol Device:C
- added D20: SS34, Diode_SMD:D_SMA, symbol Device:D_Schottky
- added J3: 12V DC center-positive, Connector_BarrelJack:BarrelJack_Wuerth_694106106102_2.0x5.5mm, symbol Connector:Barrel_Jack
- added L2: 600R@100MHz, Inductor_SMD:L_0805_2012Metric, symbol Device:FerriteBead
- added U1: AP63301WU-7, Package_TO_SOT_SMD:SOT-23-6, symbol KVM_Custom:AP63301
- C1, C4: value 47uF -> 22uF; footprint Capacitor_SMD:C_0805_2012Metric -> Capacitor_SMD:C_1206_3216Metric; Dielectric (none) -> X5R; LCSC Part (none) -> C12891; MPN (none) -> CL31A226KAHNNNE; Manufacturer (none) -> Samsung Electro-Mechanics; Sourcing (none) -> Four matched 22uF; typical DC-bias review complete; prototy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; Voltage (none) -> 25V
- C2, C5: footprint Capacitor_SMD:C_0603_1608Metric -> Capacitor_SMD:C_0805_2012Metric; Dielectric (none) -> X7R; LCSC Part (none) -> C95841; MPN (none) -> CL21B106KOQNNNE; Manufacturer (none) -> Samsung Electro-Mechanics; Voltage (none) -> 16V
- C3, C6, C7: Dielectric (none) -> X7R; LCSC Part (none) -> C131394; MPN (none) -> CC0402KRX7R9BB104; Manufacturer (none) -> YAGEO; Voltage (none) -> 50V
- L1: value 4.7uH -> 6.8uH; footprint inductor_5040:IND-SMD_L5.0-W5.0-1 -> KVM_Custom_Footprints:Bourns_SRP7050TA; LCSC Part (none) -> C2046414; MPN (none) -> SRP7050TA-6R8M; Manufacturer (none) -> Bourns; Sourcing (none) -> Manufacturer land pattern verified; assembly procurement pe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
- R1: value 750k -> 53.6k; LCSC Part (none) -> C852835; MPN (none) -> RT0402BRD0753K6L; Manufacturer (none) -> YAGEO; Power (none) -> 62.5mW; Temperature coefficient (none) -> 25ppm/C; Tolerance (none) -> 0.1%
- R2: value 100k -> 10k; LCSC Part (none) -> C190095; MPN (none) -> RT0402BRD0710KL; Manufacturer (none) -> YAGEO; Power (none) -> 62.5mW; Temperature coefficient (none) -> 25ppm/C; Tolerance (none) -> 0.1%
- U2: value AP2112K-3.3 -> AP2112K-3.3TRG1; LCSC Part (none) -> C51118; MPN (none) -> AP2112K-3.3TRG1
Connections:
- net +5V: now also R1.1, C33.1, C51.1, C52.1, L2.1; no longer C3.1, R1.2
- net +VIN: now also C3.1, C16.1, C30.1, D20.1 (K), U1.3 (VIN)
- net GND: now also C16.2, C30.2, C32.2, C51.2, C52.2, J3.2, U1.4 (GND)
- net LDO_VIN: now reaches U2.1 (VIN), U2.3 (EN)
- net LDO_VIN: now also C32.1, L2.2
- net BUCK_FB: now reaches R2.1
- net BUCK_FB: now also R1.2, C33.2, U1.1 (FB); no longer R1.1
- net BUCK_SW: now reaches L1.1
- net BUCK_SW: now also C31.2, U1.5 (SW)
- new net BUCK_BOOT: C31.1, U1.6 (BOOT)
- new net VIN_RAW: D20.2 (A), J3.1
- no-connect marks 0 -> 2
Other:
- note added: "12V input -> reverse-polarity diode -> 5V buck -> 3.3V LDO. AP63301 EN intentionally floating per Diodes. R1/R2 set nominal 5.088V. Prototype: verify 5V rail at full USB load and validate LDO temperature."
- title: PDN — Power Delivery Network -> Two-computer HDMI and USB switch
