File: sheet_stm32.kicad_sch (KiCad schematic)
At the start: 8 parts, among them SW1 SW_Push, U3 STM32F030C8Tx

Commit message: Publish A2 hardware, firmware, and verification package
Parts:
- added C27, C28, C29, C53, C54, C55: 100nF, Capacitor_SMD:C_0402_1005Metric, symbol Device:C
- added J4: SWD, Connector_PinHeader_2.54mm:PinHeader_1x05_P2.54mm_Vertical, symbol Connector_Generic:Conn_01x05
- added R23, R24, R34, R36, R38: 100k, Resistor_SMD:R_0402_1005Metric, symbol Device:R
- added R35, R37: 150k, Resistor_SMD:R_0402_1005Metric, symbol Device:R
- added R49: 10k, Resistor_SMD:R_0402_1005Metric, symbol Device:R
- added R50: 1k, Resistor_SMD:R_0402_1005Metric, symbol Device:R
- added U34: TPS3808G33DBVR, Package_TO_SOT_SMD:SOT-23-6, symbol Power_Supervisor:TPS3808DBV
- added U35: TPS3808G50DBVR, Package_TO_SOT_SMD:SOT-23-6, symbol Power_Supervisor:TPS3808DBV
- added U36: SN74LVC1G97DBVR, Package_TO_SOT_SMD:SOT-23-6, symbol KVM_Custom:SN74LVC1G97DBVR
- C8, C9: Dielectric (none) -> X7R; LCSC Part (none) -> C131394; MPN (none) -> CC0402KRX7R9BB104; Manufacturer (none) -> YAGEO; Voltage (none) -> 50V
- R11, R22: LCSC Part (none) -> C25900; MPN (none) -> 0402WGF4701TCE; Manufacturer (none) -> UNI-ROYAL; Power (none) -> 62.5mW; Tolerance (none) -> 1%
- R3, R4: LCSC Part (none) -> C25744; MPN (none) -> 0402WGF1002TCE; Manufacturer (none) -> UNI-ROYAL; Power (none) -> 62.5mW; Tolerance (none) -> 1%
- SW1: LCSC Part (none) -> C86707; MPN (none) -> B3F-4050; Manufacturer (none) -> Omron
- U3: LCSC Part (none) -> C23922; MPN (none) -> STM32F030C8T6; Manufacturer (none) -> STMicroelectronics
Connections:
- net +3.3V: now also C27.1, C28.1, C29.1, C53.1, C54.1, C55.1, J4.1 (Pin_1), U34.3 (~{MR}), U34.5 (SENSE), U34.6 (VDD), U35.3 (~{MR}), U35.6 (VDD), U36.5 (VCC)
- net GND: now also C27.2, C28.2, C29.2, C53.2, C54.2, C55.2, J4.3 (Pin_3), R23.2, R24.2, R35.2, R37.2, R38.2, R49.2, R50.2, U34.2 (GND), U35.2 (GND), U36.1 (IN1), U36.2 (GND); no longer C8.1
- net HOST_SELECT: now also R23.1
- net MUX_RESET: now also R24.1
- net MCU_NRST: now reaches C8.2, R3.2, U3.7 (NRST)
- net MCU_NRST: now also J4.5 (Pin_5), U34.1 (~{RESET}), U35.1 (~{RESET}), U36.6 (IN2)
- net HOST1_PRESENT: now reaches U3.16 (PA6)
- net HOST1_PRESENT: now also R34.2, R35.1
- net HOST2_PRESENT: now reaches U3.17 (PA7)
- net HOST2_PRESENT: now also R36.2, R37.1
- net USB_OE_N: now reaches U3.29 (PA8)
- net HUB_RESET_REQ: now reaches U3.30 (PA9)
- net HUB_RESET_REQ: now also R49.1, U36.3 (IN0)
- net HUB_VBUS_DET: now reaches U3.31 (PA10)
- net HUB_VBUS_DET: now also R38.1
- net SWDIO: now reaches U3.34 (PA13)
- net SWDIO: now also J4.2 (Pin_2)
- net SWCLK: now reaches U3.37 (PA14)
- net SWCLK: now also J4.4 (Pin_4)
- net TUSB1_SEL: no longer names the net of U3.12 (PA2)
- net TUSB2_SEL: no longer names the net of U3.11 (PA1)
- new net +5V: U35.5 (SENSE)
- new net HOST1_VBUS: R34.1
- new net HOST2_VBUS: R36.1
- new net HUB_RESET_N: U36.4 (Y)
- new net RESET_CAP_RETURN: C8.1, R50.1
- no-connect marks 32 -> 29
Other:
- note added: "Power supervision: both rails valid before MCU release; CT open = 12-28 ms delay. U35 senses +5V but is powered by +3.3V, including partial back-power conditions. U36 is a Schmitt-input AND: HUB_RESET_N = MCU_NRST AND HUB_RESET_REQ. R49 holds the firmware request low during MCU reset; PA9 remains push-pull."
- note added: "SWD header: target voltage reference only; do not power board from debugger."
- title: (none) -> Two-computer HDMI and USB switch
