File: sheet_usbc.kicad_sch (KiCad schematic)
At the start: 27 parts, among them J1 USB_C_Host_B, J2 USB_C_Host_B, U4 TUSB1046A-DCIRNQR, U5 TUSB1046A-DCIRNQR, U6 HD3SS215RTQT, U7 TUSB1064RNQT, U8 TUSB1064RNQT

Commit message: Publish A2 hardware, firmware, and verification package
Parts:
- removed C16, C17: 0.1uF, Capacitor_SMD:C_0402_1005Metric, symbol Device:C
- removed J_DP1, J_DP2: 472720001, dp_connector:CONN-SMD_472720001, symbol dp_connector:472720001
- removed U4, U5: TUSB1046A-DCIRNQR, Package_DFN_QFN:WQFN-24-1EP_4x4mm_P0.5mm_EP2.6x2.6mm_ThermalVias, symbol TUSB1046A-DCIRNQR:TUSB1046A-DCIRNQR
- removed U7, U8: TUSB1064RNQT, easyeda2kicad:WQFN-40_L6.0-W4.0-P0.40-TL-EP, symbol easyeda2kicad:TUSB1064RNQT
- added C47, C48: 100nF, Capacitor_SMD:C_0402_1005Metric, symbol Device:C
- added C49, C50: 1uF, Capacitor_SMD:C_0603_1608Metric, symbol Device:C
- added J_HDMI_C1_MON1: HDMI_A_1.4, KVM_Custom_Footprints:Assembly_J_HDMI_C1_MON1, symbol Connector:HDMI_A_1.4
- added J_HDMI_C1_MON2: HDMI_A_1.4, KVM_Custom_Footprints:Assembly_J_HDMI_C1_MON2, symbol Connector:HDMI_A_1.4
- added J_HDMI_C2_MON1: HDMI_A_1.4, KVM_Custom_Footprints:Assembly_J_HDMI_C2_MON1, symbol Connector:HDMI_A_1.4
- added J_HDMI_C2_MON2: HDMI_A_1.4, KVM_Custom_Footprints:Assembly_J_HDMI_C2_MON2, symbol Connector:HDMI_A_1.4
- added J_HDMI_MON1: HDMI_A_1.4, KVM_Custom_Footprints:Assembly_J_HDMI_MON1, symbol Connector:HDMI_A_1.4
- added J_HDMI_MON2: HDMI_A_1.4, KVM_Custom_Footprints:Assembly_J_HDMI_MON2, symbol Connector:HDMI_A_1.4
- added R19, R20: 100k, Resistor_SMD:R_0402_1005Metric, symbol Device:R
- added R43, R45: 10k, Resistor_SMD:R_0402_1005Metric, symbol Device:R
- added R44: 10k, KVM_Custom_Footprints:Assembly_R44, symbol Device:R
- added R46: 10k, KVM_Custom_Footprints:Assembly_R46, symbol Device:R
- added R47, R48: 210k, Resistor_SMD:R_0402_1005Metric, symbol Device:R
- added U11, U12, U13, U14, U15, U16, U17, U18, U19, U4, U5, U7: TPD4E02B04DQA, KVM_Custom_Footprints:USON-10_2.5x1.0mm_P0.5mm_Assembly, symbol Power_Protection:TPD4E02B04DQA
- added U24, U25, U26, U27, U28, U29, U30, U31: TPD4E05U06DQAR, KVM_Custom_Footprints:USON-10_2.5x1.0mm_P0.5mm_Assembly, symbol KVM_Custom:TPD4E05U06DQA
- added U32, U33: TPS2553DBVR, Package_TO_SOT_SMD:SOT-23-6, symbol KVM_Custom:TPS2553DBV
- added U8: HD3SS215IRTQR, Package_DFN_QFN:QFN-56-1EP_8x8mm_P0.5mm_EP4.5x5.2mm_ThermalVias, symbol HD3SS215:HD3SS215RTQT
- C10, C11, C12, C13, C14, C15: Dielectric (none) -> X7R; LCSC Part (none) -> C131394; MPN (none) -> CC0402KRX7R9BB104; Manufacturer (none) -> YAGEO; Voltage (none) -> 50V
- J1, J2: value USB_C_Host_B -> USB4105-GF-A-120; footprint KVM_Custom_Footprints:CUI_UJ31-CH-G2-SMT-TR -> Connector_USB:USB_C_Receptacle_GCT_USB4105-xx-A_16P_TopMnt_Horizontal; symbol Connector:USB_C_Receptacle -> KVM_Custom:USB4105_USB2; LCSC Part (none) -> C5184243; MPN (none) -> USB4105-GF-A-120; Sourcing (none) -> Limited stock; confirm JLC procurement quantity including a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
- R10, R7, R8, R9: LCSC Part (none) -> C25905; MPN (none) -> 0402WGF5101TCE; Manufacturer (none) -> UNI-ROYAL; Power (none) -> 62.5mW; Tolerance (none) -> 1%
- R14, R15, R16, R6: value 100k -> 47k; LCSC Part (none) -> C25792; MPN (none) -> 0402WGF4702TCE; Manufacturer (none) -> UNI-ROYAL; Power (none) -> 62.5mW; Tolerance (none) -> 1%
- R17, R18: LCSC Part (none) -> C25741; MPN (none) -> 0402WGF1003TCE; Manufacturer (none) -> UNI-ROYAL; Power (none) -> 62.5mW; Tolerance (none) -> 1%
- U6: value HD3SS215RTQT -> HD3SS215IRTQR; footprint Package_DFN_QFN:QFN-16-1EP_3x3mm_P0.5mm_EP1.7x1.7mm_ThermalVias -> Package_DFN_QFN:QFN-56-1EP_8x8mm_P0.5mm_EP4.5x5.2mm_ThermalVias; LCSC Part (none) -> C2674402; MPN (none) -> HD3SS215IRTQT; Manufacturer (none) -> Texas Instruments; Sourcing (none) -> Same device as IRTQR; TI verifies only reel size differs. J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
Connections:
- net +3.3V: now also C10.1, C11.1, C12.1, C13.1, C14.1, C15.1, R43.1, R45.1, U32.3 (EN), U33.3 (EN), U8.19 (VDD), U8.55 (VDD)
- net HOST_SELECT: now also U8.56 (Dx_SEL)
- net MUX_RESET: now also U8.43 (OE)
- net GND: now reaches C13.2
- net GND: now also C10.2, C11.2, C12.2, C14.2, C15.2, J1.A1 (GND), J1.A12 (GND), J1.B1 (GND), J1.B12 (GND), J1.SH (SHIELD), J2.A1 (GND), J2.A12 (GND), J2.B1 (GND), J2.B12 (GND), J2.SH (SHIELD), R10.2, R17.2, R18.2, R7.2, R8.2, R9.2, U6.10 (GND), U6.33 (GND), U6.36 (GND), U6.39 (GND), U6.4 (GND), U6.46 (GND), U6.49 (GND), U6.52 (GND), U6.57 (PAD), U6.7 (GND), C47.2, C48.2, C49.2, C50.2, J_HDMI_C1_MON1.11 (CKS), J_HDMI_C1_MON1.17 (GND), J_HDMI_C1_MON1.2 (D2S), J_HDMI_C1_MON1.5 (D1S), J_HDMI_C1_MON1.8 (D0S), J_HDMI_C1_MON1.SH, J_HDMI_C1_MON2.11 (CKS), J_HDMI_C1_MON2.17 (GND), J_HDMI_C1_MON2.2 (D2S), J_HDMI_C1_MON2.5 (D1S), J_HDMI_C1_MON2.8 (D0S), J_HDMI_C1_MON2.SH, J_HDMI_C2_MON1.11 (CKS), J_HDMI_C2_MON1.17 (GND), J_HDMI_C2_MON1.2 (D2S), J_HDMI_C2_MON1.5 (D1S), J_HDMI_C2_MON1.8 (D0S), J_HDMI_C2_MON1.SH, J_HDMI_C2_MON2.11 (CKS), J_HDMI_C2_MON2.17 (GND), J_HDMI_C2_MON2.2 (D2S), J_HDMI_C2_MON2.5 (D1S), J_HDMI_C2_MON2.8 (D0S), J_HDMI_C2_MON2.SH, J_HDMI_MON1.11 (CKS), J_HDMI_MON1.17 (GND), J_HDMI_MON1.2 (D2S), J_HDMI_MON1.5 (D1S), J_HDMI_MON1.8 (D0S), J_HDMI_MON1.SH, J_HDMI_MON2.11 (CKS), J_HDMI_MON2.17 (GND), J_HDMI_MON2.2 (D2S), J_HDMI_MON2.5 (D1S), J_HDMI_MON2.8 (D0S), J_HDMI_MON2.SH, R19.2, R20.2, R44.2, R46.2, R47.2, R48.2, U11.3 (G), U11.8 (G), U12.3 (G), U12.8 (G), U13.3 (G), U13.8 (G), U14.3 (G), U14.8 (G), U15.3 (G), U15.8 (G), U16.3 (G), U16.8 (G), U17.3 (G), U17.8 (G), U18.3 (G), U18.8 (G), U19.3 (G), U19.8 (G), U24.3 (G), U24.8 (G), U25.3 (G), U25.8 (G), U26.3 (G), U26.8 (G), U27.3 (G), U27.8 (G), U28.3 (G), U28.8 (G), U29.3 (G), U29.8 (G), U30.3 (G), U30.8 (G), U31.3 (G), U31.8 (G), U32.2 (GND), U33.2 (GND), U4.3 (G), U4.8 (G), U5.3 (G), U5.8 (G), U7.3 (G), U7.8 (G), U8.10 (GND), U8.33 (GND), U8.36 (GND), U8.39 (GND), U8.4 (GND), U8.46 (GND), U8.49 (GND), U8.52 (GND), U8.57 (PAD), U8.7 (GND)
- net HOST1_CC2: now reaches J1.B5 (CC2), R10.1
- net HOST1_CC2: now also U24.5 (IO4)
- net HDMI_MON1_5V: now reaches R6.2
- net HDMI_MON1_5V: now also R14.2, C49.1, J_HDMI_MON1.18 (+5V), U32.6 (OUT)
- net HOST1_CC1: now reaches J1.A5 (CC1), R9.1
- net HOST1_CC1: now also U24.4 (IO3), U24.7 (NC)
- net MON1_D0_P: now reaches U6.8 (DC2(p))
- net MON1_D0_P: now also J_HDMI_MON1.7 (D0+), U5.1 (IO1), U5.10 (NC); no longer C13.1
- net HOST2_VBUS: now reaches J2.A4 (VBUS), J2.A9 (VBUS), J2.B4 (VBUS), J2.B9 (VBUS)
- net HOST2_CC1: now reaches J2.A5 (CC1), R7.1
- net HOST2_CC1: now also U25.4 (IO3), U25.7 (NC)
- net HOST2_CC2: now reaches J2.B5 (CC2), R8.1
- net HOST2_CC2: now also U25.5 (IO4)
- net MON1_D2_P: now reaches U6.2 (DC0(p))
- net MON1_D2_P: now also J_HDMI_MON1.1 (D2+), U4.1 (IO1), U4.10 (NC); no longer C10.2
- net MON1_D0_N: now reaches U6.9 (DC2(n))
- net MON1_D0_N: now also J_HDMI_MON1.9 (D0-), U5.2 (IO2), U5.9 (NC); no longer C12.1
- net MON1_D1_N: now reaches U6.6 (DC1(n))
- net MON1_D1_N: now also J_HDMI_MON1.6 (D1-), U4.5 (IO4), U4.6 (NC); no longer C15.1
- net HDMI_MODE_1: now reaches U6.1 (AUX_SEL)
- net HDMI_MODE_1: now also R43.2, R44.1
- net MON1_D3_P: now reaches U6.11 (DC3(p))
- net MON1_D3_P: now also J_HDMI_MON1.10 (CK+), U5.4 (IO3), U5.7 (NC)
- net MON1_D3_N: now reaches U6.12 (DC3(n))
- net MON1_D3_N: now also J_HDMI_MON1.12 (CK-), U5.5 (IO4), U5.6 (NC)
- net MON1_HPD: now reaches U6.15 (HPDC)
- net MON1_HPD: now also J_HDMI_MON1.19 (HPD/HEAC-), U30.4 (IO3)
- net MON1_DDC_CLK: now reaches U6.18 (DDCCLK_C)
- net MON1_DDC_CLK: now also R6.1, J_HDMI_MON1.15 (SCL), U30.1 (IO1)
- net C2_MON1_DDC_CLK: now reaches U6.22 (DDCCLK_B)
- net C2_MON1_DDC_CLK: now also J_HDMI_C2_MON1.15 (SCL), U27.1 (IO1)
- net C2_MON1_DDC_DAT: now reaches U6.23 (DDCDAT_B)
- net C2_MON1_DDC_DAT: now also J_HDMI_C2_MON1.16 (SDA), U27.2 (IO2)
- net MON1_DDC_DAT: now reaches U6.26 (DDCDAT_C)
- net MON1_DDC_DAT: now also R14.1, J_HDMI_MON1.16 (SDA), U30.2 (IO2)
- net C1_MON1_DDC_CLK: now reaches U6.27 (DDCCLK_A)
- net C1_MON1_DDC_CLK: now also J_HDMI_C1_MON1.15 (SCL), U26.1 (IO1)
- net C1_MON1_DDC_DAT: now reaches U6.28 (DDCDAT_A)
- net C1_MON1_DDC_DAT: now also J_HDMI_C1_MON1.16 (SDA), U26.2 (IO2)
- net MON1_D2_N: now reaches U6.3 (DC0(n))
- net MON1_D2_N: now also J_HDMI_MON1.3 (D2-), U4.2 (IO2), U4.9 (NC); no longer C11.1
- net MON1_D1_P: now reaches U6.5 (DC1(p))
- net MON1_D1_P: now also J_HDMI_MON1.4 (D1+), U4.4 (IO3), U4.7 (NC); no longer C14.2
- net HDMI_MON2_5V: now reaches R16.2
- net HDMI_MON2_5V: now also R15.2, C50.1, J_HDMI_MON2.18 (+5V), U33.6 (OUT)
- net HOST1_VBUS: now reaches J1.A4 (VBUS), J1.A9 (VBUS), J1.B4 (VBUS), J1.B9 (VBUS)
- net AUXA_N: no longer names the net of U6.29 (AUXA(n))
- net AUXA_P: no longer names the net of U6.30 (AUXA(p))
- net AUXB_N: no longer names the net of U6.25 (AUXB(n))
- net AUXB_P: no longer names the net of U6.24 (AUXB(p))
- net DA0_N renamed C1_MON1_D2_N
- net C1_MON1_D2_N: now also J_HDMI_C1_MON1.3 (D2-), U12.2 (IO2), U12.9 (NC)
- net DA0_P renamed C1_MON1_D2_P
- net C1_MON1_D2_P: now also J_HDMI_C1_MON1.1 (D2+), U12.1 (IO1), U12.10 (NC)
- net DA1_N renamed C1_MON1_D1_N
- net C1_MON1_D1_N: now also J_HDMI_C1_MON1.6 (D1-), U12.5 (IO4), U12.6 (NC)
- net DA1_P renamed C1_MON1_D1_P
- net C1_MON1_D1_P: now also J_HDMI_C1_MON1.4 (D1+), U12.4 (IO3), U12.7 (NC)
- net DA2_N renamed C1_MON1_D0_N
- net C1_MON1_D0_N: now also J_HDMI_C1_MON1.9 (D0-), U13.2 (IO2), U13.9 (NC)
- net DA2_P renamed C1_MON1_D0_P
- net C1_MON1_D0_P: now also J_HDMI_C1_MON1.7 (D0+), U13.1 (IO1), U13.10 (NC)
- net DA3_N renamed C1_MON1_D3_N
- net C1_MON1_D3_N: now also J_HDMI_C1_MON1.12 (CK-), U13.5 (IO4), U13.6 (NC)
- net DA3_P renamed C1_MON1_D3_P
- net C1_MON1_D3_P: now also J_HDMI_C1_MON1.10 (CK+), U13.4 (IO3), U13.7 (NC)
- net DB0_N renamed C2_MON1_D2_N
- net C2_MON1_D2_N: now also J_HDMI_C2_MON1.3 (D2-), U14.2 (IO2), U14.9 (NC)
- net DB0_P renamed C2_MON1_D2_P
- net C2_MON1_D2_P: now also J_HDMI_C2_MON1.1 (D2+), U14.1 (IO1), U14.10 (NC)
- net DB1_N renamed C2_MON1_D1_N
- net C2_MON1_D1_N: now also J_HDMI_C2_MON1.6 (D1-), U14.5 (IO4), U14.6 (NC)
- net DB1_P renamed C2_MON1_D1_P
- net C2_MON1_D1_P: now also J_HDMI_C2_MON1.4 (D1+), U14.4 (IO3), U14.7 (NC)
- net DB2_N renamed C2_MON1_D0_N
- net C2_MON1_D0_N: now also J_HDMI_C2_MON1.9 (D0-), U15.2 (IO2), U15.9 (NC)
- net DB2_P renamed C2_MON1_D0_P
- net C2_MON1_D0_P: now also J_HDMI_C2_MON1.7 (D0+), U15.1 (IO1), U15.10 (NC)
- net DB3_N renamed C2_MON1_D3_N
- net C2_MON1_D3_N: now also J_HDMI_C2_MON1.12 (CK-), U15.5 (IO4), U15.6 (NC)
- net DB3_P renamed C2_MON1_D3_P
- net C2_MON1_D3_P: now also J_HDMI_C2_MON1.10 (CK+), U15.4 (IO3), U15.7 (NC)
- removed net EXP: J1.A1 (GND), J1.A12 (GND), J1.B1 (GND), J1.B12 (GND), J1.SH (SHIELD), J2.A1 (GND), J2.A12 (GND), J2.B1 (GND), J2.B12 (GND), J2.SH (SHIELD), R10.2, R14.1, R15.2, R16.1, R17.2, R18.1, R6.1, R7.2, R8.2, R9.2, U6.10 (GND), U6.33 (GND), U6.36 (GND), U6.39 (GND), U6.4 (GND), U6.46 (GND), U6.49 (GND), U6.52 (GND), U6.57 (PAD), U6.7 (GND)
- net HPDA renamed C1_MON1_HPD
- net C1_MON1_HPD: now also R17.1, J_HDMI_C1_MON1.19 (HPD/HEAC-), U26.4 (IO3); no longer R15.1
- net HPDB renamed C2_MON1_HPD
- net C2_MON1_HPD: now also R18.1, J_HDMI_C2_MON1.19 (HPD/HEAC-), U27.4 (IO3); no longer R17.1
- net USB2_DN_A renamed USB_HOST1_N
- net USB_HOST1_N: now also U24.2 (IO2), U24.9 (NC)
- net USB2_DN_B renamed USB_HOST2_N
- net USB_HOST2_N: now also U25.2 (IO2), U25.9 (NC)
- net USB2_DP_A renamed USB_HOST1_P
- net USB_HOST1_P: now also U24.1 (IO1), U24.10 (NC)
- net USB2_DP_B renamed USB_HOST2_P
- net USB_HOST2_P: now also U25.1 (IO1), U25.10 (NC)
- new net +5V: C47.1, C48.1, U32.1 (IN), U33.1 (IN)
- new net C1_MON2_D0_N: J_HDMI_C1_MON2.9 (D0-), U17.2 (IO2), U17.9 (NC), U8.51 (DA1(p))
- new net C1_MON2_D0_P: J_HDMI_C1_MON2.7 (D0+), U17.1 (IO1), U17.10 (NC), U8.50 (DA1(n))
- new net C1_MON2_D1_N: J_HDMI_C1_MON2.6 (D1-), U16.5 (IO4), U16.6 (NC), U8.48 (DA2(p))
- new net C1_MON2_D1_P: J_HDMI_C1_MON2.4 (D1+), U16.4 (IO3), U16.7 (NC), U8.47 (DA2(n))
- new net C1_MON2_D2_N: J_HDMI_C1_MON2.3 (D2-), U16.2 (IO2), U16.9 (NC), U8.45 (DA3(p))
- new net C1_MON2_D2_P: J_HDMI_C1_MON2.1 (D2+), U16.1 (IO1), U16.10 (NC), U8.44 (DA3(n))
- new net C1_MON2_D3_N: J_HDMI_C1_MON2.12 (CK-), U17.5 (IO4), U17.6 (NC), U8.54 (DA0(p))
- new net C1_MON2_D3_P: J_HDMI_C1_MON2.10 (CK+), U17.4 (IO3), U17.7 (NC), U8.53 (DA0(n))
- new net C1_MON2_DDC_CLK: J_HDMI_C1_MON2.15 (SCL), U28.1 (IO1), U8.27 (DDCCLK_A)
- new net C1_MON2_DDC_DAT: J_HDMI_C1_MON2.16 (SDA), U28.2 (IO2), U28.9 (NC), U8.28 (DDCDAT_A)
- new net C1_MON2_HPD: J_HDMI_C1_MON2.19 (HPD/HEAC-), R19.1, U28.4 (IO3), U8.16 (HPDA)
- new net C2_MON2_D0_N: J_HDMI_C2_MON2.9 (D0-), U19.2 (IO2), U19.9 (NC), U8.38 (DB1(p))
- new net C2_MON2_D0_P: J_HDMI_C2_MON2.7 (D0+), U19.1 (IO1), U19.10 (NC), U8.37 (DB1(n))
- new net C2_MON2_D1_N: J_HDMI_C2_MON2.6 (D1-), U18.5 (IO4), U18.6 (NC), U8.35 (DB2(p))
- new net C2_MON2_D1_P: J_HDMI_C2_MON2.4 (D1+), U18.4 (IO3), U18.7 (NC), U8.34 (DB2(n))
- new net C2_MON2_D2_N: J_HDMI_C2_MON2.3 (D2-), U18.2 (IO2), U18.9 (NC), U8.32 (DB3(p))
- new net C2_MON2_D2_P: J_HDMI_C2_MON2.1 (D2+), U18.1 (IO1), U18.10 (NC), U8.31 (DB3(n))
- new net C2_MON2_D3_N: J_HDMI_C2_MON2.12 (CK-), U19.5 (IO4), U19.6 (NC), U8.41 (DB0(p))
- new net C2_MON2_D3_P: J_HDMI_C2_MON2.10 (CK+), U19.4 (IO3), U19.7 (NC), U8.40 (DB0(n))
- new net C2_MON2_DDC_CLK: J_HDMI_C2_MON2.15 (SCL), U29.1 (IO1), U8.22 (DDCCLK_B)
- new net C2_MON2_DDC_DAT: J_HDMI_C2_MON2.16 (SDA), U29.2 (IO2), U8.23 (DDCDAT_B)
- new net C2_MON2_HPD: J_HDMI_C2_MON2.19 (HPD/HEAC-), R20.1, U29.4 (IO3), U8.17 (HPDB)
- new net HDMI_ILIM1: R47.1, U32.5 (ILIM)
- new net HDMI_ILIM2: R48.1, U33.5 (ILIM)
- new net HDMI_MODE_2: R45.2, R46.1, U8.1 (AUX_SEL)
- new net MON2_D0_N: J_HDMI_MON2.9 (D0-), U11.2 (IO2), U11.9 (NC), U8.5 (DC1(p))
- new net MON2_D0_P: J_HDMI_MON2.7 (D0+), U11.1 (IO1), U11.10 (NC), U8.6 (DC1(n))
- new net MON2_D1_N: J_HDMI_MON2.6 (D1-), U7.5 (IO4), U7.6 (NC), U8.8 (DC2(p))
- new net MON2_D1_P: J_HDMI_MON2.4 (D1+), U7.4 (IO3), U7.7 (NC), U8.9 (DC2(n))
- new net MON2_D2_N: J_HDMI_MON2.3 (D2-), U7.2 (IO2), U7.9 (NC), U8.11 (DC3(p))
- new net MON2_D2_P: J_HDMI_MON2.1 (D2+), U7.1 (IO1), U7.10 (NC), U8.12 (DC3(n))
- new net MON2_D3_N: J_HDMI_MON2.12 (CK-), U11.5 (IO4), U11.6 (NC), U8.2 (DC0(p))
- new net MON2_D3_P: J_HDMI_MON2.10 (CK+), U11.4 (IO3), U11.7 (NC), U8.3 (DC0(n))
- new net MON2_DDC_CLK: J_HDMI_MON2.15 (SCL), R15.1, U31.1 (IO1), U8.18 (DDCCLK_C)
- new net MON2_DDC_DAT: J_HDMI_MON2.16 (SDA), R16.1, U31.2 (IO2), U8.26 (DDCDAT_C)
- new net MON2_HPD: J_HDMI_MON2.19 (HPD/HEAC-), U31.4 (IO3), U8.15 (HPDC)
- no-connect marks 55 -> 71
Other:
- note added: "External-port ESD: 5.5V-rated arrays on USB D+/D-/CC and HDMI DDC/HPD. TPD4E02B04 arrays remain on the eight TMDS conductors of each HDMI connector."
- note added: "HDMI input pin 18 rails are isolated from board +5V and from each other."
- note added: "HDMI mode: AUX_SEL must be VDD/2. 10k/10k dividers; never leave AUX_SEL floating (TI datasheet section 7.5)."
- title: (none) -> Two-computer HDMI and USB switch
- moved on the sheet: R10, R7, R8, R9
